File: USBChargerT1_AAMU-Hope/USBChargerT1_AAMU-HOPE.kicad_sch (KiCad schematic)
At the start: 40 parts, among them J2 USB CONN, J3 USB CONN, U1 LM73606RNPT, U2 TPS2549RTER, U3 TPS2549RTER

Commit message: Finish Schematics and fully functional
I updated the schematics from U1 (LM73606) to U1 (LM73605), which made the schematics work from the previous results of LM73606. Also, the download to symbol and footprint LM73605 is attached. I also attached the symbol editor picture of U1 Pins (LM73605).
Parts:
- removed J3: USB CONN, UJ2-AH-1-SMT:CUI_UJ2-AH-1-SMT, symbol Senior Design:UJ2-AH-1-SMT
- removed U1: LM73606RNPT, LM73606RNPT:QFN50P600X400X80-31N, symbol Senior Design:LM73606RNPT
- added J1: USB CONN, UJ2-AH-1-SMT:CUI_UJ2-AH-1-SMT, symbol Senior Design:UJ2-AH-1-SMT
- added U1: LM73605QRNPTQ1, RNP0030A, symbol Senior Design:LM73605QRNPTQ1
- L1: value 6 SuH -> 6.8uH
- R11: value 200K -> 20K
Connections:
- net +12V: now also C19.1, U1.18 (EN), U1.20 (VIN), U1.21 (VIN), U1.22 (VIN), U1.7 (VCC)
- net CS: now also R8.1, R9.1
- net FB: now also U1.11 (FB)
- net GND: now also J1.4 (GND), J1.5, J1.6, U1.12 (NC), U1.13 (NC), U1.14 (NC), U1.15 (NC), U1.16 (PGOOD), U1.19 (AGND), U1.23 (PGND), U1.24 (PGND), U1.25 (PGND), U1.26 (PGND), U1.27 (NC), U1.28 (NC), U1.29 (NC), U1.30 (NC), U1.31 (DAP)
- net SW: now also U1.1 (SW), U1.2 (SW), U1.3 (SW), U1.4 (SW), U1.5 (SW)
- net VOUT: now also C14.1, C15.1, C16.1, R3.2, U2.1 (IN), U2.5 (EN), U3.1 (IN), U3.5 (EN), U1.8 (BIAS)
- net at C18.1, U3.12 (OUT): now also J2.1 (VBUS)
- net at R4.1: now also U1.17 (SYNC)
- net at R2.1: now also U1.9 (RT)
- net at C1.1: now also U1.6 (CBOOT)
- net at C17.1, U2.12 (OUT): now also J1.1 (VBUS); no longer J2.1 (VBUS)
- net B_D+: now reaches U2.10 (DP_IN)
- net B_D+: now also J2.3 (D+), U3.10 (DP_IN), J1.3 (D+)
- net B_D-: now reaches U2.11 (DM_IN)
- net B_D-: now also J2.2 (D-), U3.11 (DM_IN), J1.2 (D-)
- net DIM: now reaches R12.1, R13.1

Commit message: Finished Project
I ran the DRC(Design Rule Check) on board; everything is wired properly and checks well with no errors.  Changed the pad properties on U1, U2, and U3 to SMD Aperture. Also, I changed pads located with U1, U2, and U3 to SMD, too.
Parts:
- C1, C10, C11, C12, C13, C14, C15, C16, C17, C18, C19, C2, C3, C4, C5, C6, C7, C8, C9: footprint (none) -> Capacitor_SMD:C_0603_1608Metric_Pad1.08x0.95mm_HandSolder
- D1, D2: footprint (none) -> Diode_SMD:D_0603_1608Metric_Pad1.05x0.95mm_HandSolder
- J1, J2: footprint UJ2-AH-1-SMT:CUI_UJ2-AH-1-SMT -> AAMU Senior Design 2024-25:CUI_UJ2-AH-1-SMT
- L1: footprint (none) -> Inductor_SMD:L_0603_1608Metric_Pad1.05x0.95mm_HandSolder
- R1, R10, R11, R12, R13, R2, R3, R4, R5, R6, R7, R8, R9: footprint (none) -> Resistor_SMD:R_0603_1608Metric_Pad0.98x0.95mm_HandSolder
- U1: footprint RNP0030A -> AAMU Senior Design 2024-25:RNP0030A
- U2, U3: footprint RTE0016C -> AAMU Senior Design 2024-25:RTE0016C
Changed lines of the file:
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@@
 			)
 		)
-		(property "Footprint" ""
+		(property "Footprint" "Capacitor_SMD:C_0603_1608Metric_Pad1.08x0.95mm_HandSolder"
 			(at 310.8452 120.65 0)
 			(effects
@@
 			)
 		)
-		(property "Footprint" ""
+		(property "Footprint" "Capacitor_SMD:C_0603_1608Metric_Pad1.08x0.95mm_HandSolder"
 			(at 171.1452 110.49 0)
 			(effects
@@
 			)
 		)
-		(property "Footprint" ""
+		(property "Footprint" "Resistor_SMD:R_0603_1608Metric_Pad0.98x0.95mm_HandSolder"
 			(at 413.766 120.904 90)
 			(effects
@@
 			)
 		)
-		(property "Footprint" ""
+		(property "Footprint" "Capacitor_SMD:C_0603_1608Metric_Pad1.08x0.95mm_HandSolder"
 			(at 367.9952 120.65 0)
 			(effects
@@
 			)
 		)
-		(property "Footprint" ""
+		(property "Footprint" "Capacitor_SMD:C_0603_1608Metric_Pad1.08x0.95mm_HandSolder"
 			(at 157.1752 110.49 0)
 			(effects
@@
 			)
 		)
-		(property "Footprint" ""
+		(property "Footprint" "Capacitor_SMD:C_0603_1608Metric_Pad1.08x0.95mm_HandSolder"
 			(at 394.6652 120.65 0)
 			(effects
@@
 			)
 		)
-		(property "Footprint" ""
+		(property "Footprint" "Capacitor_SMD:C_0603_1608Metric_Pad1.08x0.95mm_HandSolder"
 			(at 381.9652 120.65 0)
 			(effects
@@
 			)
 		)
-		(property "Footprint" "RTE0016C"
+		(property "Footprint" "AAMU Senior Design 2024-25:RTE0016C"
 			(at 172.72 264.16 0)
 			(effects
@@
 			)
 		)
-		(property "Footprint" ""
+		(property "Footprint" "Capacitor_SMD:C_0603_1608Metric_Pad1.08x0.95mm_HandSolder"
 			(at 144.4752 110.49 0)
 			(effects
@@
 			)
 		)
-		(property "Footprint" ""
+		(property "Footprint" "Capacitor_SMD:C_0603_1608Metric_Pad1.08x0.95mm_HandSolder"
 			(at 277.8252 104.14 0)
 			(effects
@@
 			)
 		)
-		(property "Footprint" ""
+		(property "Footprint" "Resistor_SMD:R_0603_1608Metric_Pad0.98x0.95mm_HandSolder"
 			(at 413.766 138.684 90)
 			(effects
@@
 			)
 		)
-		(property "Footprint" ""
+		(property "Footprint" "Resistor_SMD:R_0603_1608Metric_Pad0.98x0.95mm_HandSolder"
 			(at 209.296 120.396 90)
 			(effects
@@
 			)
 		)
-		(property "Footprint" ""
+		(property "Footprint" "Inductor_SMD:L_0603_1608Metric_Pad1.05x0.95mm_HandSolder"
 			(at 295.91 106.68 0)
 			(effects
@@
 			)
 		)
-		(property "Footprint" ""
+		(property "Footprint" "Capacitor_SMD:C_0603_1608Metric_Pad1.08x0.95mm_HandSolder"
 			(at 366.7252 267.97 0)
 			(effects
@@
 			)
 		)
-		(property "Footprint" ""
+		(property "Footprint" "Capacitor_SMD:C_0603_1608Metric_Pad1.08x0.95mm_HandSolder"
 			(at 224.4852 260.35 0)
 			(effects
@@
 			)
 		)
-		(property "Footprint" ""
+		(property "Footprint" "Diode_SMD:D_0603_1608Metric_Pad1.05x0.95mm_HandSolder"
 			(at 486.41 129.54 0)
 			(effects
@@
 			)
 		)
-		(property "Footprint" ""
+		(property "Footprint" "Capacitor_SMD:C_0603_1608Metric_Pad1.08x0.95mm_HandSolder"
 			(at 280.3652 138.43 0)
 			(effects
@@
 			)
 		)
-		(property "Footprint" "RTE0016C"
+		(property "Footprint" "AAMU Senior Design 2024-25:RTE0016C"
 			(at 425.45 273.05 0)
 			(effects
@@
 			)
 		)
-		(property "Footprint" ""
+		(property "Footprint" "Resistor_SMD:R_0603_1608Metric_Pad0.98x0.95mm_HandSolder"
 			(at 475.234 128.524 90)
 			(effects
@@
 			)
 		)
-		(property "Footprint" ""
+		(property "Footprint" "Capacitor_SMD:C_0603_1608Metric_Pad1.08x0.95mm_HandSolder"
 			(at 338.7852 120.65 0)
 			(effects
@@
 			)
 		)
-		(property "Footprint" ""
+		(property "Footprint" "Capacitor_SMD:C_0603_1608Metric_Pad1.08x0.95mm_HandSolder"
 			(at 430.2252 120.65 0)
 			(effects
@@
 			)
 		)
-		(property "Footprint" ""
+		(property "Footprint" "Resistor_SMD:R_0603_1608Metric_Pad0.98x0.95mm_HandSolder"
 			(at 209.296 125.476 90)
 			(effects
@@
 			)
 		)
-		(property "Footprint" ""
+		(property "Footprint" "Resistor_SMD:R_0603_1608Metric_Pad0.98x0.95mm_HandSolder"
 			(at 413.766 159.004 90)
 			(effects
@@
 			)
 		)
-		(property "Footprint" ""
+		(property "Footprint" "Capacitor_SMD:C_0603_1608Metric_Pad1.08x0.95mm_HandSolder"
 			(at 324.8152 120.65 0)
 			(effects
@@
 			)
 		)
-		(property "Footprint" ""
+		(property "Footprint" "Resistor_SMD:R_0603_1608Metric_Pad0.98x0.95mm_HandSolder"
 			(at 465.836 274.574 90)
 			(effects
@@
 			)
 		)
-		(property "Footprint" "UJ2-AH-1-SMT:CUI_UJ2-AH-1-SMT"
+		(property "Footprint" "AAMU Senior Design 2024-25:CUI_UJ2-AH-1-SMT"
 			(at 510.54 251.46 0)
 			(effects
@@
 			)
 		)
-		(property "Footprint" ""
+		(property "Footprint" "Resistor_SMD:R_0603_1608Metric_Pad0.98x0.95mm_HandSolder"
 			(at 289.306 122.936 90)
 			(effects
@@
 			)
 		)
-		(property "Footprint" ""
+		(property "Footprint" "Capacitor_SMD:C_0603_1608Metric_Pad1.08x0.95mm_HandSolder"
 			(at 477.2152 269.24 0)
 			(effects
@@
 			)
 		)
-		(property "Footprint" ""
+		(property "Footprint" "Capacitor_SMD:C_0603_1608Metric_Pad1.08x0.95mm_HandSolder"
 			(at 354.0252 120.65 0)
 			(effects
@@
 			)
 		)
-		(property "Footprint" ""
+		(property "Footprint" "Resistor_SMD:R_0603_1608Metric_Pad0.98x0.95mm_HandSolder"
 			(at 213.106 265.684 90)
 			(effects
@@
 			)
 		)
-		(property "Footprint" "RNP0030A"
+		(property "Footprint" "AAMU Senior Design 2024-25:RNP0030A"
 			(at 242.57 121.92 0)
 			(effects
@@
 			)
 		)
-		(property "Footprint" ""
+		(property "Footprint" "Resistor_SMD:R_0603_1608Metric_Pad0.98x0.95mm_HandSolder"
 			(at 139.954 263.144 90)
 			(effects
@@
 			)
 		)
-		(property "Footprint" ""
+		(property "Footprint" "Resistor_SMD:R_0603_1608Metric_Pad0.98x0.95mm_HandSolder"
 			(at 475.234 117.094 90)
 			(effects
@@
 			)
 		)
-		(property "Footprint" "UJ2-AH-1-SMT:CUI_UJ2-AH-1-SMT"
+		(property "Footprint" "AAMU Senior Design 2024-25:CUI_UJ2-AH-1-SMT"
 			(at 257.81 242.57 0)
 			(effects
@@
 			)
 		)
-		(property "Footprint" ""
+		(property "Footprint" "Diode_SMD:D_0603_1608Metric_Pad1.05x0.95mm_HandSolder"
 			(at 486.41 118.11 0)
 			(effects
@@
 			)
 		)
-		(property "Footprint" ""
+		(property "Footprint" "Capacitor_SMD:C_0603_1608Metric_Pad1.08x0.95mm_HandSolder"
 			(at 113.9952 259.08 0)
 			(effects
@@
 			)
 		)
-		(property "Footprint" ""
+		(property "Footprint" "Resistor_SMD:R_0603_1608Metric_Pad0.98x0.95mm_HandSolder"
 			(at 430.276 138.684 90)
 			(effects
@@
 			)
 		)
-		(property "Footprint" ""
+		(property "Footprint" "Capacitor_SMD:C_0603_1608Metric_Pad1.08x0.95mm_HandSolder"
 			(at 183.8452 110.49 0)
 			(effects
@@
 			)
 		)
-		(property "Footprint" ""
+		(property "Footprint" "Capacitor_SMD:C_0603_1608Metric_Pad1.08x0.95mm_HandSolder"
 			(at 199.0852 115.57 0)
 			(effects
@@
 			)
 		)
-		(property "Footprint" ""
+		(property "Footprint" "Resistor_SMD:R_0603_1608Metric_Pad0.98x0.95mm_HandSolder"
 			(at 392.684 272.034 90)
 			(effects
